File: hardware/afe.kicad_sch (KiCad schematic)
At the start: 35 parts, among them J2 Conn_01x02_Pin, U2 MCP6002-xMC, U3 4052

Commit message: started PCB routing, AFE ready, rest still in Progress
Parts:
- removed TP6, TP7: TestPoint, TestPoint:TestPoint_Pad_D1.5mm, symbol Connector:TestPoint
- C5: renamed from C4; value 91p -> 82p
- U2: Reichelt Part-Number MCP 6002-I/SN -> (none)
- renumbered C1 to C2, C2 to C3, C3 to C4, C5 to C6, C6 to C7, C7 to C8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
Other:
- note added: "offset voltage buffer"
- note removed: "offset voltage"
