File: hardware/parallax.kicad_pcb (KiCad board)
At the start: 2 copper layers, 102 parts, among them J1 Conn_Coaxial, J2 Conn_Coaxial, J3 Conn_Coaxial, J4 Conn_01x10_Pin, J5 Conn_01x02_Pin, J6 Conn_01x02_Pin, J7 Conn_01x02_Pin, SW1 SW_Push_Dual, U1 Pico, U2 MCP6002-xMC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

Commit message: Hardware: now in the state where a testing prototype can be ordered
Parts:
- removed SW1: SW_Push_Dual, work:SW_PUSH-12mm
- added SW2: SW_Push, Button_Switch_THT:SW_PUSH_6mm_H4.3mm, F.Cu at (205.5, 49.8)
- moved R2 74.3 mm to (175.5, 37.3), turned to -90 degrees
- moved D2 72.3 mm to (175.6, 40.7), turned to -90 degrees
- moved R51 64.1 mm to (137.0, 61.5), turned to -90 degrees
- moved C18 63.6 mm to (137.9, 50.5)
- moved R3 61.4 mm to (202.8, 49.0), turned to -90 degrees
- moved R4 58.7 mm to (202.0, 54.2), turned to 180 degrees
- moved TP7 58.3 mm to (139.2, 59.3)
- moved TP6 58.3 mm to (140.0, 45.5)
- moved D1 54.0 mm to (175.2, 59.6), turned to 90 degrees
- moved C1 49.3 mm to (198.8, 53.5), turned to -90 degrees
- moved R1 48.4 mm to (175.2, 63.1), turned to 90 degrees
- moved U6 44.7 mm to (138.0, 53.5), turned to 180 degrees
- moved C19 41.7 mm to (138.0, 56.5), turned to 0 degrees
- moved R41 41.2 mm to (146.8, 51.2), turned to 180 degrees
- moved J3 41.2 mm to (136.2, 69.1), turned to 180 degrees
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- renumbered TP19 to TP6, TP20 to TP7
Connections:
- C19 pad 1: +5V -> +3V3
- U6 pad 5: +5V -> +3V3
Routing:
- net +3V3: track 12.1 -> 259.5 mm, vias 0 -> 4
- net Reset: track 0.00 -> 48.9 mm
- net LED_2: track 0.00 -> 46.0 mm
- net Net-(U6-+): track 0.00 -> 24.6 mm
- net /Analog Front-End/analog_in: track 3.21 -> 16.9 mm
- net GND: track 5.84 -> 17.7 mm, vias 7 -> 81
- net Net-(U6--): track 0.00 -> 11.8 mm
- net /Analog Front-End1/analog_in: track 3.21 -> 13.6 mm
- net Net-(R4-Pad1): track 0.00 -> 9.18 mm
- net /R2R-DAC/AWG_OUT: track 0.00 -> 6.80 mm
- net Net-(J5-Pin_2): track 0.00 -> 6.22 mm
- net Net-(R40-Pad2): track 0.00 -> 5.74 mm
- net Net-(R36-Pad2): track 0.00 -> 5.43 mm
- net /R2R-DAC/B2: track 0.00 -> 5.03 mm
- net Net-(R37-Pad2): track 0.00 -> 4.81 mm
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Other:
- board outline added: 89.9 x 52.3 mm
- board text added: "Raspberry Pi Pico with Analog Front-End"
