File: hardware/parallax.kicad_sch (KiCad schematic)
At the start: 14 parts, among them J1 Conn_Coaxial, J2 Conn_Coaxial, J3 Conn_Coaxial, J4 Conn_01x10_Pin, J5 Conn_01x02_Pin, SW1 SW_Push_Dual, U1 Pico

Commit message: Hardware: now in the state where a testing prototype can be ordered
Parts:
- removed SW1: SW_Push_Dual, work:SW_PUSH-12mm, symbol Switch:SW_Push_Dual
- added SW2: SW_Push, Button_Switch_THT:SW_PUSH_6mm_H4.3mm, symbol Switch:SW_Push
Connections:
- net Reset: now also SW2.1
- net at R4.1: now also SW2.2
Other:
- moved on the sheet: R4
Changed lines of the file:
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@@
-	)
-	(junction
-		(at 255.27 143.51)
-		(diameter 0)
-		(color 0 0 0 0)
-	)
-	(junction
-		(at 265.43 148.59)
-		(diameter 0)
-		(color 0 0 0 0)
 	)
 	(junction
@@
 	(wire
 		(pts
-			(xy 255.27 143.51) (xy 255.27 148.59)
-		)
-		(stroke
-			(width 0)
-			(type default)
-		)
-	)
-	(wire
-		(pts
 			(xy 72.39 86.36) (xy 76.2 86.36)
 		)
@@
 		(pts
 			(xy 212.09 97.79) (xy 218.44 97.79)
-		)
-		(stroke
-			(width 0)
-			(type default)
-		)
-	)
-	(wire
-		(pts
-			(xy 265.43 143.51) (xy 265.43 148.59)
 		)
 		(stroke
@@
 	(symbol
 		(lib_id "Device:R")
-		(at 269.24 148.59 90)
+		(at 269.24 143.51 90)
 		(unit 1)
 		(exclude_from_sim no)
@@
 		(fields_autoplaced yes)
 		(property "Reference" "R4"
-			(at 269.24 142.24 90)
+			(at 269.24 137.16 90)
 			(effects
 				(font
@@
 		)
 		(property "Value" "1K"
-			(at 269.24 144.78 90)
+			(at 269.24 139.7 90)
 			(effects
 				(font
@@
 		)
 		(property "Footprint" "Resistor_SMD:R_0603_1608Metric"
-			(at 269.24 150.368 90)
+			(at 269.24 145.288 90)
 			(effects
 				(font
@@
 		)
 		(property "Datasheet" "~"
-			(at 269.24 148.59 0)
+			(at 269.24 143.51 0)
 			(effects
 				(font
@@
 		)
 		(property "Description" "Resistor"
-			(at 269.24 148.59 0)
+			(at 269.24 143.51 0)
 			(effects
 				(font
@@
 	(symbol
 		(lib_id "power:GND")
-		(at 273.05 148.59 0)
+		(at 273.05 143.51 0)
 		(unit 1)
 		(exclude_from_sim no)
@@
 		(dnp no)
 		(property "Reference" "#PWR026"
-			(at 273.05 154.94 0)
+			(at 273.05 149.86 0)
 			(effects
 				(font
@@
 		)
 		(property "Value" "GND"
-			(at 276.606 150.368 0)
+			(at 276.606 145.288 0)
 			(effects
 				(font
@@
 		)
 		(property "Footprint" ""
-			(at 273.05 148.59 0)
+			(at 273.05 143.51 0)
 			(effects
 				(font
@@
 		)
 		(property "Datasheet" ""
-			(at 273.05 148.59 0)
+			(at 273.05 143.51 0)
 			(effects
 				(font
@@
 		)
 		(property "Description" "Power symbol creates a global label with name \"GND\" , ground"
-			(at 273.05 148.59 0)
+			(at 273.05 143.51 0)
 			(effects
 				(font
@@
 	)
 	(symbol
-		(lib_id "Switch:SW_Push_Dual")
-		(at 260.35 146.05 0)
-		(unit 1)
-		(exclude_from_sim no)
-		(in_bom yes)
-		(on_board yes)
-		(dnp no)
-		(fields_autoplaced yes)
-		(property "Reference" "SW1"
-			(at 260.35 135.89 0)
-			(effects
-				(font
-					(size 1.27 1.27)
-				)
-			)
-		)
-		(property "Value" "SW_Push_Dual"
-			(at 260.35 138.43 0)
-			(effects
-				(font
-					(size 1.27 1.27)
-				)
-			)
-		)
-		(property "Footprint" "work:SW_PUSH-12mm"
-			(at 260.35 138.43 0)
-			(effects
-				(font
-					(size 1.27 1.27)
-				)
-				(hide yes)
-			)
-		)
-		(property "Datasheet" "~"
-			(at 260.35 146.05 0)
-			(effects
-				(font
-					(size 1.27 1.27)
-				)
-				(hide yes)
-			)
-		)
-		(property "Description" "Push button switch, generic, symbol, four pins"
-			(at 260.35 146.05 0)
-			(effects
-				(font
-					(size 1.27 1.27)
-				)
-				(hide yes)
-			)
-		)
-		(pin "1"
-		)
-		(pin "4"
-		)
-		(pin "2"
-		)
-		(pin "3"
-		)
-		(instances
-			(project "parallax"
-				(path "/9be75e04-ffa7-400b-a6f6-98cbc4c2c88c"
-					(reference "SW1")
-					(unit 1)
-				)
-			)
-		)
-	)
-	(symbol
 		(lib_id "power:GND")
 		(at 218.44 85.09 0)
@@
 					(unit 1)
 				)
+			)
+		)
+	)
+	(symbol
+		(lib_id "Switch:SW_Push")
+		(at 260.35 143.51 0)
+		(unit 1)
+		(exclude_from_sim no)
+		(in_bom yes)
+		(on_board yes)
+		(dnp no)
+		(fields_autoplaced yes)
+		(property "Reference" "SW2"
+			(at 260.35 135.89 0)
+			(effects
+				(font
+					(size 1.27 1.27)
+				)
+			)
+		)
+		(property "Value" "SW_Push"
+			(at 260.35 138.43 0)
+			(effects
+				(font
+					(size 1.27 1.27)
+				)
+			)
+		)
+		(property "Footprint" "Button_Switch_THT:SW_PUSH_6mm_H4.3mm"
+			(at 260.35 138.43 0)
+			(effects
+				(font
+					(size 1.27 1.27)
+				)
+				(hide yes)
+			)
+		)
+		(property "Datasheet" "~"
+			(at 260.35 138.43 0)
+			(effects
+				(font
+					(size 1.27 1.27)
+				)
+				(hide yes)
+			)
+		)
+		(property "Description" "Push button switch, generic, two pins"
+			(at 260.35 143.51 0)
+			(effects
+				(font
+					(size 1.27 1.27)
+				)
+				(hide yes)
+			)
+		)
+		(pin "1"
+		)
+		(pin "2"
+		)
+		(instances
+			(project ""
+				(path "/9be75e04-ffa7-400b-a6f6-98cbc4c2c88c"
+					(reference "SW2")
+					(unit 1)
+				)
